Commit message: certain changes where made to turtlebot - was to add the echo sim using 3D LIDAR - adding the batbot

File: turtlebot_description/urdf/sensors/astra.urdf.xacro (robot description, xacro)
@@ -4,5 +4,7 @@
   <xacro:include filename="$(find turtlebot_description)/urdf/turtlebot_properties.urdf.xacro"/>
   <!-- Xacro properties -->
-  <xacro:property name="astra_cam_py" value="-0.0125"/>
+  <xacro:property name="astra_cam_px" value="-0.129"/>
+  <xacro:property name="astra_cam_py" value="0.008"/>
+  <xacro:property name="astra_cam_pz" value="0.281"/>
   <xacro:property name="astra_depth_rel_rgb_py" value="0.0250" />
   <xacro:property name="astra_cam_rel_rgb_py"   value="-0.0125" />
@@ -11,5 +13,5 @@
   <xacro:macro name="sensor_astra" params="parent">
     <joint name="camera_rgb_joint" type="fixed">
-      <origin xyz="${cam_px} ${astra_cam_py} ${cam_pz}"
+      <origin xyz="${astra_cam_px} ${astra_cam_py} ${astra_cam_pz}"
               rpy="0 0 0"/>
       <parent link="${parent}"/>
@@ -31,5 +33,5 @@
     <link name="camera_link">
       <visual>
-        <origin xyz="-0.04 0.02 -0.01" rpy="${M_PI/2} 0 ${M_PI/2}"/>
+        <origin xyz="0 0 0" rpy="${M_PI/2} 0 ${M_PI/2}"/>
         <geometry>
           <mesh filename="package://turtlebot_description/meshes/sensors/astra.dae" scale="${astra_dae_display_scale} ${astra_dae_display_scale} ${astra_dae_display_scale}"/>

File: turtlebot_description/urdf/sensors/r200.urdf.xacro (robot description, xacro)
@@ -74,7 +74,7 @@
       <origin xyz="${r200_cam_offset_px} ${r200_cam_offset_py} ${r200_cam_offset_pz}" rpy="0 0 0"/>
       <parent link="bracket"/>
-      <child link="camera_link" />
+      <child link="camera" />
     </joint>
-    <link name="camera_link">
+    <link name="camera">
       <visual>
        <origin xyz="0 0 0" rpy="${M_PI/2} 0 ${M_PI/2}"/>
@@ -103,5 +103,5 @@
     <joint name="camera_rgb_joint" type="fixed">
       <origin xyz="${r200_cam_rgb_px} ${r200_cam_rgb_py} ${r200_cam_rgb_pz}" rpy="0 0 0"/>
-      <parent link="camera_link"/>
+      <parent link="camera"/>
       <child link="camera_rgb_frame" />
     </joint>

File: turtlebot_description/urdf/turtlebot_gazebo.urdf.xacro (robot description, xacro)
@@ -10,6 +10,6 @@
           <horizontal_fov>${60.0*M_PI/180.0}</horizontal_fov>
           <image>
-            <format>B8G8R8</format>
-            <width>640</width>
+            <format>R8G8B8</format>
+            <width>480</width>
             <height>480</height>
           </image>

File: turtlebot_description/urdf/turtlebot_properties.urdf.xacro (robot description, xacro)
@@ -19,9 +19,10 @@
      (currently in development and awaiting feedback)
    -->
-	<xacro:property name="cam_px" value="-0.087" />
+	<xacro:property name="cam_px" value="0.1" />
 <!--	<xacro:property name="cam_py" value="-0.0125" /> Y varies for different configurations. get sets in sensors_urdf -->
-	<xacro:property name="cam_pz" value="0.2870" />
+  <xacro:property name="cam_py" value="0" />
+	<xacro:property name="cam_pz" value="0.6" />
 	<xacro:property name="cam_or" value="0" />
-	<xacro:property name="cam_op" value="0" />
+	<xacro:property name="cam_op" value="0.6" />
 	<xacro:property name="cam_oy" value="0" />
 </robot>
